File: MCU-Datalogger-with-512K-EEPROM-and-Clock.kicad_pcb (KiCad board)
At the start: 2 copper layers, 0 parts

Commit message: uploaded page setting; restarting the board design
Parts:
- added BT1: Battery, Connector_PinHeader_2.54mm:PinHeader_1x02_P2.54mm_Vertical, F.Cu at (178.1, 143.5)
- added C1: 0.1uF, Capacitor_SMD:C_0805_2012Metric, F.Cu at (194.0, 139.7)
- added C2: 22pF, Capacitor_SMD:C_0805_2012Metric, F.Cu at (207.3, 156.8)
- added C3: 22pF, Capacitor_SMD:C_0805_2012Metric, F.Cu at (197.8, 139.7)
- added C4: 0.1uF, Capacitor_SMD:C_0805_2012Metric, F.Cu at (207.3, 153.7)
- added C5: 100nF, Capacitor_SMD:C_0805_2012Metric, F.Cu at (201.6, 139.7)
- added D1: LED, LED_SMD:LED_0805_2012Metric, F.Cu at (210.5, 139.7)
- added D2: LED, LED_SMD:LED_0805_2012Metric, F.Cu at (206.7, 139.7)
- added J1: Conn_01x04_Pin, Connector_PinHeader_2.54mm:PinHeader_1x04_P2.54mm_Vertical, F.Cu at (216.9, 149.8)
- added J2: Conn_01x04_Pin, Connector_PinHeader_2.54mm:PinHeader_1x04_P2.54mm_Vertical, F.Cu at (203.5, 161.3)
- added J3: Conn_01x09_Pin, Connector_PinHeader_2.54mm:PinHeader_1x09_P2.54mm_Vertical, F.Cu at (178.1, 161.3)
- added J4: Conn_02x03_Odd_Even, Connector_PinHeader_2.54mm:PinHeader_2x03_P2.54mm_Vertical, F.Cu at (214.3, 140.3)
- added R1: 10K, Resistor_SMD:R_0805_2012Metric, F.Cu at (183.9, 158.1)
- added R2: 10K, Resistor_SMD:R_0805_2012Metric, F.Cu at (187.7, 158.1)
- added R3: 4.7K, Resistor_SMD:R_0805_2012Metric, F.Cu at (206.2, 149.2)
- added R4: 4.7K, Resistor_SMD:R_0805_2012Metric, F.Cu at (206.1, 146.7)
- added R5: 330, Resistor_SMD:R_0805_2012Metric, F.Cu at (210.5, 144.1)
- added R6: 10K, Resistor_SMD:R_0805_2012Metric, F.Cu at (210.5, 146.7)
- added R7: 330, Resistor_SMD:R_0805_2012Metric, F.Cu at (206.1, 144.1)
- added U1: 24LC1025, Package_SO:SOIC-8_5.3x5.3mm_P1.27mm, F.Cu at (185.8, 140.3)
- added U2: 24LC1025, Package_SO:SOIC-8_5.3x5.3mm_P1.27mm, F.Cu at (185.8, 147.3)
- added U3: ATMEGA328P-AU, ATMEGA328P-AU:QFP80P900X900X120-32N, F.Cu at (197.2, 147.3)
- added U4: DS1337S_, DS1337S_:SOIC127P600X175-8N, F.Cu at (185.8, 154.3)
- added Y1: 32.768 KHz, Crystal:Crystal_SMD_5032-2Pin_5.0x3.2mm_HandSoldering, F.Cu at (178.1, 154.3)
- added Y2: 16 MHz, Crystal:Crystal_SMD_5032-2Pin_5.0x3.2mm_HandSoldering, F.Cu at (196.6, 154.9)
Routing:
- net /Vcc: track 0.00 -> 91.8 mm
- net GND: track 0.00 -> 72.4 mm, vias 0 -> 2
- net /SCL: track 0.00 -> 64.5 mm
- net Net-(BT1-+): track 0.00 -> 60.1 mm, vias 0 -> 3
- net /SDA: track 0.00 -> 35.1 mm
- net /D2: track 0.00 -> 29.7 mm, vias 0 -> 1
- net /D3: track 0.00 -> 26.5 mm, vias 0 -> 2
- net /TX: track 0.00 -> 26.0 mm, vias 0 -> 1
- net Net-(U3-PB7): track 0.00 -> 24.4 mm, vias 0 -> 2
- net /D4: track 0.00 -> 23.7 mm, vias 0 -> 3
- net /RX: track 0.00 -> 23.5 mm, vias 0 -> 1
- net /MOSI: track 0.00 -> 23.5 mm, vias 0 -> 1
- net Net-(U3-PB6): track 0.00 -> 20.4 mm
- net /RESET: track 0.00 -> 20.4 mm, vias 0 -> 2
- net /MISO: track 0.00 -> 19.4 mm, vias 0 -> 1
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- added copper zone on F.Cu, net /Vcc
- added copper zone on B.Cu, net GND
