File: Connectors.kicad_sch (KiCad schematic)
At the start: 4 parts, among them J1 Conn_01x04_Pin, J2 Conn_01x04_Pin, J3 Conn_01x09_Pin, J4 Conn_02x03_Odd_Even

Commit message: uploaded page setting; restarting the board design
Other:
- company: University of Notre Dame | Udemy -> ${company_name}
- title: Connectors -> Connectors : ${project_name}
Changed lines of the file:
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@@
 	(paper "A4")
 	(title_block
-		(title "Connectors")
+		(title "Connectors : ${project_name}")
 		(date "2025-07-05")
 		(rev "1.0")
-		(company "University of Notre Dame | Udemy")
-		(comment 1 "Made by Andres Perez")
+		(company "${company_name}")
+		(comment 1 "${comment_1}")
 	)
 	(hierarchical_label "D3"

Commit message: fixed schematic sck vs scl nets
Connections:
- net SCL: no longer J4.3 (Pin_3)
- new net SCK: J4.3 (Pin_3)
Changed lines of the file:
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@@
 		)
 	)
-	(hierarchical_label "SCL"
+	(hierarchical_label "SCK"
 		(shape passive)
 		(at 45.72 48.26 180)
